Commit message: camera funzionante nella simulazione :) (ci ho perso un anno di vita)

File: ros2_create3_sim/src/create3_sim/irobot_create_common/irobot_create_description/urdf/create3.urdf.xacro (robot description, xacro)
@@ -8,4 +8,5 @@
   <xacro:include filename="$(find irobot_create_description)/urdf/sensors/imu.urdf.xacro" />
   <xacro:include filename="$(find irobot_create_description)/urdf/sensors/ir_intensity.urdf.xacro" />
+  <xacro:include filename="$(find irobot_create_description)/urdf/sensors/camera_sensor.urdf.xacro" />
   <xacro:include filename="$(find irobot_create_description)/urdf/sensors/ir_opcode_receivers.urdf.xacro" />
   <xacro:include filename="$(find irobot_create_description)/urdf/sensors/optical_mouse.urdf.xacro"/>
@@ -133,4 +134,8 @@
     <origin xyz="0.1015 0.087 ${-0.055 + base_link_z_offset}" rpy="0 0 ${-pi/4}"/>
   </xacro:optical_mouse>
+  <!--Camera sensor -->
+  <xacro:camera_sensor name="front" gazebo="$(arg gazebo)" namespace="$(arg namespace)">
+    <origin xyz="0.12 0 ${0.18 + base_link_z_offset}" rpy="0 0 0"/>
+  </xacro:camera_sensor>
   <!-- Cliffs sensors -->
   <xacro:property name="cliff_z"  value="${-4.5*cm2m}" />
@@ -260,8 +265,6 @@
     <gazebo>
       <plugin filename="libgz-sim-contact-system.so" name="gz::sim::systems::Contact"></plugin>
-    </gazebo>
-    <gazebo>
       <plugin filename="libgz-sim-sensors-system.so" name="gz::sim::systems::Sensors">
-        <render_engine>ogre</render_engine>
+        <render_engine>ogre2</render_engine>
       </plugin>
     </gazebo>

Commit message: sensori di prossimita funzionanti

File: ros2_create3_sim/src/create3_sim/irobot_create_common/irobot_create_description/urdf/create3.urdf.xacro (robot description, xacro)
@@ -9,4 +9,5 @@
   <xacro:include filename="$(find irobot_create_description)/urdf/sensors/ir_intensity.urdf.xacro" />
   <xacro:include filename="$(find irobot_create_description)/urdf/sensors/camera_sensor.urdf.xacro" />
+  <xacro:include filename="$(find irobot_create_description)/urdf/sensors/ultrasonic_sensor.urdf.xacro" />
   <xacro:include filename="$(find irobot_create_description)/urdf/sensors/ir_opcode_receivers.urdf.xacro" />
   <xacro:include filename="$(find irobot_create_description)/urdf/sensors/optical_mouse.urdf.xacro"/>
@@ -138,4 +139,17 @@
     <origin xyz="0.12 0 ${0.18 + base_link_z_offset}" rpy="0 0 0"/>
   </xacro:camera_sensor>
+  <!-- Ultrasonic sensors -->
+  <!-- Front ultrasonic sensor -->
+  <xacro:ultrasonic_sensor name="front" gazebo="$(arg gazebo)" namespace="$(arg namespace)" visualize="true">
+    <origin xyz="0.14 0 ${0.05 + base_link_z_offset}" rpy="0 0 0"/>
+  </xacro:ultrasonic_sensor>
+  <!-- Left ultrasonic sensor -->
+  <xacro:ultrasonic_sensor name="front_left" gazebo="$(arg gazebo)" namespace="$(arg namespace)" visualize="true">
+    <origin xyz="0.10 0.10 ${0.05 + base_link_z_offset}" rpy="0 0 ${pi/4}"/>
+  </xacro:ultrasonic_sensor>
+  <!-- Right ultrasonic sensor -->
+  <xacro:ultrasonic_sensor name="front_right" gazebo="$(arg gazebo)" namespace="$(arg namespace)" visualize="true">
+    <origin xyz="0.10 -0.10 ${0.05 + base_link_z_offset}" rpy="0 0 ${-pi/4}"/>
+  </xacro:ultrasonic_sensor>
   <!-- Cliffs sensors -->
   <xacro:property name="cliff_z"  value="${-4.5*cm2m}" />
